Commit message: 修复：以八推进器中心分配六轴力并校正手动方向
采用实际 URDF 安装位置和中心参考系，按确认方向逐轴映射，保证单轴正负一档四路有效起步；同步发送入口并补充模型、中心平移和伪串口验证。

File: internal/underwater_description/urdf/underwater_robot.urdf (robot description, URDF)
Before this commit: robot UnderWater-Robot-ROS2, 1 links, 0 joints
Links:
- added link thruster_center
Joints:
- added joint base_to_thruster_center: type fixed, parent base_link, child thruster_center, origin xyz=-0.012873 0 -0.040532 rpy=0 0 0
